File: sky-ruler/sky-ruler.sch (KiCad schematic (older format))
At the start: 19 parts

Commit message: Updated KiCAD files
Parts:
- removed C?: 220n, symbol Device:C_Small
- removed C?: 100n, symbol Device:C_Small
- removed U?: MCP1700-3302E_SOT23, Package_TO_SOT_SMD:SOT-23, symbol Regulator_Linear:MCP1700-3302E_SOT23
- added C1, C2, C3: 100n, Capacitor_SMD:C_0805_2012Metric, symbol Device:C_Small
- added J4: PROGRAMMER, Connector_PinHeader_2.54mm:PinHeader_1x06_P2.54mm_Vertical, symbol Connector_Generic:Conn_01x06
- C4, C5: renamed from C?; footprint (none) -> Capacitor_THT:C_Disc_D3.0mm_W1.6mm_P2.50mm
- C6, C7: renamed from C?; footprint (none) -> Capacitor_SMD:C_0805_2012Metric
- D1: renamed from D?; footprint (none) -> Diode_THT:D_DO-15_P2.54mm_Vertical_AnodeUp
- J1: renamed from J?; footprint (none) -> Connector_PinHeader_2.54mm:PinHeader_1x02_P2.54mm_Vertical
- J2, J3: renamed from J?; footprint (none) -> Connector_PinHeader_2.54mm:PinHeader_1x04_P2.54mm_Vertical
- R1, R2, R3: renamed from R?; footprint (none) -> Resistor_THT:R_Axial_DIN0204_L3.6mm_D1.6mm_P5.08mm_Horizontal
- SW1, SW2: renamed from SW?; footprint (none) -> Button_Switch_THT:SW_PUSH_6mm_H4.3mm
- U2: renamed from U?; footprint Package_TO_SOT_THT:TO-220-3_Vertical -> Package_TO_SOT_THT:TO-220F-3_Horizontal_TabDown
- Y1: renamed from Y?; footprint (none) -> Crystal:Crystal_HC18-U_Vertical
- gave numbers to parts that had none: 1
Connections:
- net +5V: now also J2.4 (Pin_4), J3.3 (Pin_3), C1.2, C2.2, C3.2, J4.5 (Pin_5)
- net GND: now also J2.3 (Pin_3), J3.4 (Pin_4), C1.1, C2.1, C3.1, J4.6 (Pin_6)
- net SCL: now also J2.2 (Pin_2), J3.2 (Pin_2)
- net SDA: now also J2.1 (Pin_1), J3.1 (Pin_1)
- net RESET: now reaches R1.2, SW1.1 (A), U1.1 (~RESET~/PC6)
- net RESET: now also J4.4 (Pin_4)
- net 17_MOSI: now reaches U1.17 (PB3)
- net 17_MOSI: now also J4.1 (Pin_1)
- net 18_MISO: now reaches U1.18 (PB4)
- net 18_MISO: now also J4.2 (Pin_2)
- net 19_SCK: now reaches R3.1, U1.19 (PB5)
- net 19_SCK: now also J4.3 (Pin_3)
- no-connect marks 6 -> 14
Other:
- moved on the sheet: C4, C5, D1, R3, Y1
